File: particle_sensor_pcb/particle_sensor_pcb.kicad_pcb (KiCad board)
At the start: 2 copper layers, 71 x 74 mm, 22 parts, among them J1 USB_B_Micro, J2 PMS7003, U1 AMS1117-3.3, U2 004-0-0053, U3 DHT11, U4 ESP-12F

Commit message: Changed micro usb to Type-C port.
Parts:
- removed J1: USB_B_Micro, Connector_USB:USB_Micro-B_Amphenol_10103594-0001LF_Horizontal
- added P1: USB_C_Plug_USB2.0, Connector_USB:USB_C_Receptacle_HRO_TYPE-C-31-M-12, F.Cu at (69.0, 104.0)
- added R6: 5.1K, Resistor_SMD:R_0805_2012Metric_Pad1.20x1.40mm_HandSolder, F.Cu at (61.0, 102.0)
- added R7: 5.1K, Resistor_SMD:R_0805_2012Metric_Pad1.20x1.40mm_HandSolder, F.Cu at (61.0, 104.0)
Connections:
- J2 pad 5: Net-(J2-Pad5) -> unconnected-(J2-Pad5)
- J2 pad 6: Net-(J2-Pad6) -> unconnected-(J2-Pad6)
- J2 pad 7: Net-(J2-Pad7) -> unconnected-(J2-Pad7)
- J2 pad 8: Net-(J2-Pad8) -> unconnected-(J2-Pad8)
- U2 pad 3: Net-(U2-Pad3) -> unconnected-(U2-Pad3)
- U2 pad 4: Net-(U2-Pad4) -> unconnected-(U2-Pad4)
- U2 pad 5: Net-(U2-Pad5) -> unconnected-(U2-Pad5)
- U2 pad 6: Net-(U2-Pad6) -> unconnected-(U2-Pad6)
- U2 pad 9: Net-(U2-Pad9) -> unconnected-(U2-Pad9)
- U3 pad 3: Net-(U3-Pad3) -> unconnected-(U3-Pad3)
- U4 pad 10: Net-(U4-Pad10) -> unconnected-(U4-Pad10)
- U4 pad 11: Net-(U4-Pad11) -> unconnected-(U4-Pad11)
- U4 pad 12: Net-(U4-Pad12) -> unconnected-(U4-Pad12)
- U4 pad 13: Net-(U4-Pad13) -> unconnected-(U4-Pad13)
- U4 pad 14: Net-(U4-Pad14) -> unconnected-(U4-Pad14)
- U4 pad 16: Net-(U4-Pad16) -> unconnected-(U4-Pad16)
- U4 pad 2: Net-(U4-Pad2) -> unconnected-(U4-Pad2)
- U4 pad 21: Net-(U4-Pad21) -> unconnected-(U4-Pad21)
- U4 pad 22: Net-(U4-Pad22) -> unconnected-(U4-Pad22)
- U4 pad 9: Net-(U4-Pad9) -> unconnected-(U4-Pad9)
Routing:
- net GND: track 42.3 -> 56.0 mm
- net Net-(P1-PadB5): track 0.00 -> 11.2 mm
- net +5V: track 161.2 -> 170.1 mm
- net Net-(P1-PadA5): track 0.00 -> 7.54 mm
- removed copper zone on F.Cu, net GND
Other:
- net class Default removed
- net class Powa removed
