File: particle_sensor_pcb/particle_sensor_pcb.kicad_pcb (KiCad board)
At the start: 2 copper layers, 71 x 74 mm, 22 parts, among them J1 USB_B_Micro, J2 PMS7003, U1 AMS1117-3.3, U2 004-0-0053, U3 DHT11, U4 ESP-12F

Commit message: USB-C connector, fix bodge, add jumper board
Parts:
- removed MH1, MH2, MH3: MountingHole_2.2mm_M2, MountingHole:MountingHole_2.2mm_M2
- added J3: PMS7003, Connector_PinSocket_1.27mm:PinSocket_2x05_P1.27mm_Vertical, F.Cu at (108.2, 69.4)
- added P1: USB_C_, lib:TYPE-C-31-M-17_handsolder, F.Cu at (68.1, 104.6)
- added R6: 1M, Resistor_SMD:R_0805_2012Metric_Pad1.20x1.40mm_HandSolder, F.Cu at (60.9, 102.6)
- added R7: 12K, Resistor_SMD:R_0805_2012Metric_Pad1.20x1.40mm_HandSolder, F.Cu at (59.9, 93.0)
- added R8: 12K, Resistor_SMD:R_0805_2012Metric_Pad1.20x1.40mm_HandSolder, F.Cu at (59.9, 90.9)
- added R9: 12K, Resistor_SMD:R_0805_2012Metric_Pad1.20x1.40mm_HandSolder, F.Cu at (71.9, 57.1)
- added REF**: MountingHole_2.2mm_M2, MountingHole:MountingHole_2.2mm_M2, F.Cu at (111.0, 53.3)
- added REF**: MountingHole_2.2mm_M2, MountingHole:MountingHole_2.2mm_M2, F.Cu at (106.4, 53.3)
- added REF**: MountingHole_2.2mm_M2, MountingHole:MountingHole_2.2mm_M2, F.Cu at (109.0, 40.0)
- added REF**: MountingHole_2.2mm_M2, MountingHole:MountingHole_2.2mm_M2, F.Cu at (103.4, 53.3)
- added REF**: MountingHole_2.2mm_M2, MountingHole:MountingHole_2.2mm_M2, F.Cu at (105.7, 53.3)
- added REF**: MountingHole_2.2mm_M2, MountingHole:MountingHole_2.2mm_M2, F.Cu at (114.0, 53.3)
- added REF**: MountingHole_2.2mm_M2, MountingHole:MountingHole_2.2mm_M2, F.Cu at (101.1, 53.3)
- added REF**: MountingHole_2.2mm_M2, MountingHole:MountingHole_2.2mm_M2, F.Cu at (110.2, 53.3)
- added REF**: MountingHole_2.2mm_M2, MountingHole:MountingHole_2.2mm_M2, F.Cu at (104.1, 53.3)
- added REF**: MountingHole_2.2mm_M2, MountingHole:MountingHole_2.2mm_M2, F.Cu at (104.9, 53.3)
- added REF**: MountingHole_2.2mm_M2, MountingHole:MountingHole_2.2mm_M2, F.Cu at (108.0, 53.3)
- added REF**: MountingHole_2.2mm_M2, MountingHole:MountingHole_2.2mm_M2, F.Cu at (112.5, 53.3)
- added REF**: MountingHole_2.2mm_M2, MountingHole:MountingHole_2.2mm_M2, F.Cu at (111.8, 53.3)
- added REF**: MountingHole_2.2mm_M2, MountingHole:MountingHole_2.2mm_M2, F.Cu at (109.5, 53.3)
- added REF**: MountingHole_2.2mm_M2, MountingHole:MountingHole_2.2mm_M2, F.Cu at (60.0, 98.0)
- added REF**: MountingHole_2.2mm_M2, MountingHole:MountingHole_2.2mm_M2, F.Cu at (102.6, 53.3)
- added REF**: MountingHole_2.2mm_M2, MountingHole:MountingHole_2.2mm_M2, F.Cu at (101.9, 53.3)
- added REF**: MountingHole_2.2mm_M2, MountingHole:MountingHole_2.2mm_M2, F.Cu at (60.0, 40.0)
- added REF**: MountingHole_2.2mm_M2, MountingHole:MountingHole_2.2mm_M2, F.Cu at (113.3, 53.3)
- added REF**: MountingHole_2.2mm_M2, MountingHole:MountingHole_2.2mm_M2, F.Cu at (107.2, 53.3)
- added REF**: MountingHole_2.2mm_M2, MountingHole:MountingHole_2.2mm_M2, F.Cu at (108.7, 53.3)
- J1: value USB_B_Micro -> DST_JUMP; footprint Connector_USB:USB_Micro-B_Amphenol_10103594-0001LF_Horizontal -> Connector_PinHeader_2.54mm:PinHeader_2x05_P2.54mm_Vertical
- J2: value PMS7003 -> SRC_JUMP
- moved J1 63.3 mm to (112.5, 55.8), turned to -90 degrees
Connections:
- J1 pad 1: +5V -> +5V_JMP
- J1 pad 2: Net-(J1-Pad2) -> +5V_JMP
- J1 pad 3: Net-(J1-Pad3) -> GND_JMP
- J1 pad 4: Net-(J1-Pad4) -> GND_JMP
- J1 pad 5: GND -> unconnected-(J1-Pad5)
- J1 pad 6: GND -> unconnected-(J1-Pad6)
- J2 pad 5: Net-(J2-Pad5) -> unconnected-(J2-Pad5)
- J2 pad 6: Net-(J2-Pad6) -> unconnected-(J2-Pad6)
- J2 pad 7: Net-(J2-Pad7) -> unconnected-(J2-Pad7)
- J2 pad 8: Net-(J2-Pad8) -> unconnected-(J2-Pad8)
- U2 pad 3: Net-(U2-Pad3) -> unconnected-(U2-Pad3)
- U2 pad 4: Net-(U2-Pad4) -> unconnected-(U2-Pad4)
- U2 pad 5: Net-(U2-Pad5) -> unconnected-(U2-Pad5)
- U2 pad 6: Net-(U2-Pad6) -> unconnected-(U2-Pad6)
- U2 pad 9: Net-(U2-Pad9) -> unconnected-(U2-Pad9)
- U3 pad 3: Net-(U3-Pad3) -> unconnected-(U3-Pad3)
- U4 pad 10: Net-(U4-Pad10) -> unconnected-(U4-Pad10)
- U4 pad 11: Net-(U4-Pad11) -> unconnected-(U4-Pad11)
- U4 pad 12: Net-(U4-Pad12) -> unconnected-(U4-Pad12)
- U4 pad 13: Net-(U4-Pad13) -> unconnected-(U4-Pad13)
- U4 pad 14: Net-(U4-Pad14) -> unconnected-(U4-Pad14)
- U4 pad 2: Net-(U4-Pad2) -> unconnected-(U4-Pad2)
- U4 pad 21: Net-(U4-Pad21) -> unconnected-(U4-Pad21)
- U4 pad 22: Net-(U4-Pad22) -> unconnected-(U4-Pad22)
- U4 pad 9: Net-(U4-Pad9) -> unconnected-(U4-Pad9)
Routing:
- net /SHIELD: track 0.00 -> 18.5 mm
- net +5V_JMP: track 0.00 -> 15.7 mm
- net D1_JMP: track 0.00 -> 15.2 mm
- net /CC2: track 0.00 -> 12.7 mm
- net /CC1: track 0.00 -> 10.6 mm
- net D2_JMP: track 0.00 -> 10.4 mm
- net GND: track 42.3 -> 32.9 mm, vias 16 -> 13
- net +5V: track 161.2 -> 167.2 mm
- net Net-(U4-Pad16): track 0.00 -> 5.07 mm
- added copper zone on B.Cu, net GND_JMP
- added copper zone on F.Cu, net GND_JMP
Other:
- outline, holes or cut-outs redrawn
- net class Default removed
- net class Powa removed
